Commit message: update main

File: PI/src/mason_control/urdf/mason.ros2_control.xacro (robot description, xacro)
@@ -6,13 +6,18 @@
         <hardware>
           <plugin>mason_hardware/MasonInterface</plugin>
-          <param name="device">/dev/ttyACM0</param>
           <param name="left_motor_name">MotorJointLeft</param>
           <param name="right_motor_name">MotorJointRight</param>
           <param name="horizontal_motor_name">MotorTop</param>
+          <param name="device">/dev/ttyACM0</param>
           <param name="baud_rate">115200</param>
-          <!-- <param name="timeout_ms">50</param> -->
+          <param name="timeout_ms">50</param>
           <param name="id_left">0</param>
           <param name="id_right">1</param>
           <param name="id_horizontal">1</param>
+          <!-- <param name="example_param_hw_start_duration_sec">0.0</param>
+          <param name="example_param_hw_stop_duration_sec">3.0</param>
+          <param name="example_param_hw_slowdown">${slowdown}</param> -->
+          <!-- <param name="direction_right">0</param>
+          <param name="direction_left">0</param> -->
         </hardware>
       </xacro:unless>
@@ -23,4 +28,14 @@
         </hardware>
       </xacro:if>
+      <!-- <joint name="MotorJointLeft">
+        <state_interface name="position"/>
+        <state_interface name="velocity"/>
+        <command_interface name="velocity"/>
+      </joint>
+      <joint name="MotorJointRight">
+        <state_interface name="position"/>
+        <state_interface name="velocity"/>
+        <command_interface name="velocity"/>
+      </joint> -->
       <joint name="${prefix}MotorJointLeft">
         <command_interface name="position">
@@ -28,5 +43,5 @@
           <param name="max">1</param>
         </command_interface>
-        <!-- <command_interface name="velocity">
+        <command_interface name="velocity">
           <param name="min">-1</param>
           <param name="max">1</param>
@@ -35,8 +50,8 @@
           <param name="min">-1</param>
           <param name="max">1</param>
-        </command_interface> -->
+        </command_interface>
         <state_interface name="position"/>
-        <!-- <state_interface name="velocity"/>
-        <state_interface name="acceleration"/> -->
+        <state_interface name="velocity"/>
+        <state_interface name="acceleration"/>
       </joint>
       <joint name="${prefix}MotorTop">
@@ -45,5 +60,5 @@
           <param name="max">1</param>
         </command_interface>
-        <!-- <command_interface name="velocity">
+        <command_interface name="velocity">
           <param name="min">-1</param>
           <param name="max">1</param>
@@ -52,8 +67,8 @@
           <param name="min">-1</param>
           <param name="max">1</param>
-        </command_interface> -->
+        </command_interface>
         <state_interface name="position"/>
-        <!-- <state_interface name="velocity"/>
-        <state_interface name="acceleration"/> -->
+        <state_interface name="velocity"/>
+        <state_interface name="acceleration"/>
       </joint>
     </ros2_control>

File: PI/src/mason_control/urdf/mason_description.urdf.xacro (robot description, xacro)
@@ -2496,8 +2496,7 @@
         <pose>0.8 0 0.5 0 0 0</pose>
       </frame> -->
-    <!-- Rotate 90 degrees (π/2) about the X-axis -->
-    <!-- <gazebo reference="tof_link">
+    <gazebo reference="tof_link">
         <sensor name="tof_sensor" type="gpu_lidar">
-          <pose>0 0 0 1.570796 0 0</pose>
+          <pose>0 0 0 1.570796 0 0</pose> <!-- Rotate 90 degrees (π/2) about the X-axis -->
           <update_rate>10</update_rate>
           <topic>tof_sensor</topic>
@@ -2526,5 +2525,5 @@
           <visualize>true</visualize>
         </sensor>
-      </gazebo> -->
+      </gazebo>
     <!-- Contact sensors bottom right -->
     <link name="contact_sensor_bottom_right">
@@ -2709,5 +2708,5 @@
         rpy="0 0 0" />
     </joint>
-    <!-- <gazebo reference="contact_sensor_bottom_right">
+    <gazebo reference="contact_sensor_bottom_right">
       <sensor name="bottom_right_contact_sensor" type="contact">
         <collision>Bottom Right Collision</collision>
@@ -2738,5 +2737,5 @@
         <collision>Middle Left Collision</collision>
       </sensor>
-    </gazebo> -->
+    </gazebo>
     <link name="imu_link"></link>
     <joint name="gearbox_to_imu" type="fixed">
@@ -2744,5 +2743,5 @@
       <child link="imu_link"></child>
     </joint>
-    <!-- <gazebo reference="imu_link">
+    <gazebo reference="imu_link">
       <sensor name="gearbox_imu" type="imu">
         <always_on>1</always_on>
@@ -2772,5 +2771,5 @@
       </sensor>
     </gazebo>
-    <gazebo>
+    <!-- <gazebo>
       <plugin filename="gz_ros2_control-system" name="gz_ros2_control::GazeboSimROS2ControlPlugin">
         <parameters>$(find mason_description)/description/config/mason.yaml</parameters>

File: PI/src/mason_description/description/urdf/mason.urdf.xacro (robot description, xacro)
@@ -3,8 +3,8 @@
   <xacro:arg name="use_mock_hardware" default="false" />
   <xacro:arg name="slowdown" default="100.0" />
-  <xacro:include filename="$(find mason_description)/description/mason_description.urdf.xacro" />
-  <xacro:include filename="$(find mason_description)/description/mason.ros2_control.xacro" />
+  <xacro:include filename="$(find mason_description)/description/urdf/mason_description.urdf.xacro" />
+  <xacro:include filename="$(find mason_description)/description/urdf/mason.ros2_control.xacro" />
   <xacro:mason />
   <xacro:mason_ros2_control
-    name="MasonRos2Control" prefix="" slowdown="$(arg slowdown)" use_mock_hardware="$(arg use_mock_hardware)"/>
+    name="MasonHardware" prefix="" slowdown="$(arg slowdown)" use_mock_hardware="$(arg use_mock_hardware)"/>
 </robot>
