Commit message: fix write thread

File: PI/install/mason_description/share/mason_description/description/urdf/mason.ros2_control.xacro (robot description, xacro)
@@ -7,9 +7,8 @@
           <plugin>mason_hardware/MasonInterface</plugin>
           <param name="device">/dev/ttyACM0</param>
-          <param name="left_motor_name">MotorJointLeft</param>
-          <param name="right_motor_name">MotorJointRight</param>
-          <param name="horizontal_motor_name">MotorTop</param>
+          <param name="left_motor_name">motor_left</param>
+          <param name="right_motor_name">motor_right</param>
+          <param name="horizontal_motor_name">motor_horizontal</param>
           <param name="baud_rate">115200</param>
-          <!-- <param name="timeout_ms">50</param> -->
           <param name="id_left">125</param>
           <param name="id_right">72</param>
@@ -23,37 +22,13 @@
         </hardware>
       </xacro:if>
-      <joint name="${prefix}MotorTop">
+      <joint name="${prefix}motor_horizontal">
         <command_interface name="position">
-          <param name="min">-1</param>
-          <param name="max">1</param>
         </command_interface>
-        <!-- <command_interface name="velocity">
-          <param name="min">-1</param>
-          <param name="max">1</param>
+        <state_interface name="position"/>
+      </joint>
+      <joint name="${prefix}motor_left">
+        <command_interface name="position">
         </command_interface>
-        <command_interface name="acceleration">
-          <param name="min">-1</param>
-          <param name="max">1</param>
-        </command_interface> -->
-        <state_interface name="position"/>
-        <!-- <state_interface name="velocity"/> -->
-        <!-- <state_interface name="acceleration"/> -->
-      </joint>
-      <joint name="${prefix}MotorJointLeft">
-        <command_interface name="position">
-          <param name="min">-1</param>
-          <param name="max">1</param>
-        </command_interface>
-        <!-- <command_interface name="velocity">
-          <param name="min">-1</param>
-          <param name="max">1</param>
-        </command_interface>
-        <command_interface name="acceleration">
-          <param name="min">-1</param>
-          <param name="max">1</param>
-        </command_interface> -->
-        <state_interface name="position"/>
-        <!-- <state_interface name="velocity"/> -->
-        <!-- <state_interface name="acceleration"/> -->
+        <state_interface name="position"/>>
       </joint>
     </ros2_control>

File: PI/install/mason_description/share/mason_description/description/urdf/mason_description.urdf.xacro (robot description, xacro)
@@ -3,2778 +3,22 @@
   <xacro:macro name="mason">
     <link name="world" />
-    <link
-      name="RightBar">
-      <inertial>
-        <origin
-          xyz="-1.34046800536292 -0.272459904837881 0.0490096577850858"
-          rpy="0 0 0" />
-        <mass
-          value="5.55312910017424" />
-        <inertia
-          ixx="0.782838152186612"
-          ixy="1.21611266476934E-17"
-          ixz="-4.49093050475392E-19"
-          iyy="0.782838152186612"
-          iyz="-4.74065607624699E-17"
-          izz="0.00154494115749392" />
-      </inertial>
-      <visual>
-        <origin
-          xyz="0 0 0"
-          rpy="0 0 0" />
-        <geometry>
-          <mesh
-            filename="$(find mason_description)/description/meshes/RightBar.STL" />
-        </geometry>
-        <material
-          name="">
-          <color
-            rgba="0.647058823529412 0.619607843137255 0.588235294117647 1" />
-        </material>
-      </visual>
-      <collision>
-        <origin
-          xyz="0 0 0"
-          rpy="0 0 0" />
-        <geometry>
-          <mesh
-            filename="$(find mason_description)/description/meshes/RightBar.STL" />
-        </geometry>
-      </collision>
-    </link>
-    <joint name="world_to_rightBar" type="fixed">
-      <origin rpy="0 0 0" xyz="0 0 0" />
-      <parent link="world" />
-      <child link="RightBar" />
+    <link name="right_bar"> </link>
+    <link name="left_bar"> </link>
+    <link name="horizontal_bar"> </link>
+    <joint name="motor_left" type="continuous">
+      <parent link="world"/>
+      <child link="left_bar"/>
+      <axis xyz="0 0 1"/>
     </joint>
-    <link
-      name="RightBracketTop">
-      <inertial>
-        <origin
-          xyz="-0.0307068750932176 0.0431985153087461 -6.29781428340692E-07"
-          rpy="0 0 0" />
-        <mass
-          value="0.000214749814862541" />
-        <inertia
-          ixx="5.04014900228215E-07"
-          ixy="1.41838418654998E-07"
-          ixz="-1.26884314163884E-12"
-          iyy="2.49863376560336E-07"
-          iyz="4.06202656032707E-12"
-          izz="5.24669847054164E-07" />
-      </inertial>
-      <visual>
-        <origin
-          xyz="0 0 0"
-          rpy="0 0 0" />
-        <geometry>
-          <mesh
-            filename="$(find mason_description)/description/meshes/RightBracketTop.STL" />
-        </geometry>
-        <material
-          name="">
-          <color
-            rgba="0.4 0.4 0.4 1" />
-        </material>
-      </visual>
-      <collision>
-        <origin
-          xyz="0 0 0"
-          rpy="0 0 0" />
-        <geometry>
-          <mesh
-            filename="$(find mason_description)/description/meshes/RightBracketTop.STL" />
-        </geometry>
-      </collision>
-    </link>
-    <joint
-      name="RBT_RB"
-      type="fixed">
-      <origin
-        xyz="-1.43796800536526 -0.392459904838281 0.589966540848759"
-        rpy="-3.14159265358979 0 3.14159265358979" />
-      <parent
-        link="RightBar" />
-      <child
-        link="RightBracketTop" />
-      <axis
-        xyz="0 0 0" />
+    <joint name="motor_right" type="continuous">
+      <parent link="world"/>
+      <child link="right_bar"/>
+      <axis xyz="0 0 1"/>
     </joint>
-    <link
-      name="RightBracketBottom">
-      <inertial>
-        <origin
-          xyz="-0.0307095280172158 0.0432034395198194 4.9852419820029E-07"
-          rpy="0 0 0" />
-        <mass
-          value="0.214769503083403" />
-        <inertia
-          ixx="0.000504017787094408"
-          ixy="0.000141840084805534"
-          ixz="-2.55519874076561E-09"
-          iyy="0.000249864733012362"
-          iyz="5.55018450253158E-09"
-          izz="0.000524673250439356" />
-      </inertial>
-      <visual>
-        <origin
-          xyz="0 0 0"
-          rpy="0 0 0" />
-        <geometry>
-          <mesh
-            filename="$(find mason_description)/description/meshes/RightBracketBottom.STL" />
-        </geometry>
-        <material
-          name="">
-          <color
-            rgba="0.792156862745098 0.819607843137255 0.933333333333333 1" />
-        </material>
-      </visual>
-      <collision>
-        <origin
-          xyz="0 0 0"
-          rpy="0 0 0" />
-        <geometry>
-          <mesh
-            filename="$(find mason_description)/description/meshes/RightBracketBottom.STL" />
-        </geometry>
-      </collision>
-    </link>
-    <joint
-      name="RBB_RB"
-      type="fixed">
-      <origin
-        xyz="-1.43796800536388 -0.392459904837929 -0.437021328543411"
-        rpy="-3.14159265358979 0 3.14159265358979" />
-      <parent
-        link="RightBar" />
-      <child
-        link="RightBracketBottom" />
-      <axis
-        xyz="0 0 0" />
+    <joint name="motor_horizontal" type="continuous">
+      <parent link="world"/>
+      <child link="horizontal_bar"/>
+      <axis xyz="0 0 1"/>
     </joint>
-    <link
-      name="LeftBar">
-      <inertial>
-        <origin
-          xyz="6.93889390390723E-17 0.65 5.55111512312578E-17"
-          rpy="0 0 0" />
-        <mass
-          value="5.55312910017434" />
-        <inertia
-          ixx="0.782838152186632"
-          ixy="-3.84480360700148E-18"
-          ixz="-1.03516199438847E-17"
-          iyy="0.00154494115749394"
-          iyz="-1.94626228426363E-18"
-          izz="0.782838152186632" />
-      </inertial>
-      <visual>
-        <origin
-          xyz="0 0 0"
-          rpy="0 0 0" />
-        <geometry>
-          <mesh
-            filename="$(find mason_description)/description/meshes/LeftBar.STL" />
-        </geometry>
-        <material
-          name="">
-          <color
-            rgba="0.647058823529412 0.619607843137255 0.588235294117647 1" />
-        </material>
-      </visual>
-      <collision>
-        <origin
-          xyz="0 0 0"
-          rpy="0 0 0" />
-        <geometry>
-          <mesh
-            filename="$(find mason_description)/description/meshes/LeftBar.STL" />
-        </geometry>
-      </collision>
-    </link>
-    <joint
-      name="LB_RB"
-      type="fixed">
-      <origin
-        xyz="-0.0824680053628981 -0.272459904837888 -0.600990342214936"
-        rpy="1.5707963267949 0 0" />
-      <parent
-        link="RightBar" />
-      <child
-        link="LeftBar" />
-      <axis
-        xyz="0 0 0" />
-    </joint>
-    <link
-      name="LeftBracketTop">
-      <inertial>
-        <origin
-          xyz="-0.0307068750922646 0.0431985153087082 -6.29781428118648E-07"
-          rpy="0 0 0" />
-        <mass
-          value="0.000214749814862542" />
-        <inertia
-          ixx="5.04014900228219E-07"
-          ixy="1.41838418654999E-07"
-          ixz="-1.26884314002485E-12"
-          iyy="2.49863376560337E-07"
-          iyz="4.06202656005297E-12"
-          izz="5.24669847054167E-07" />
-      </inertial>
-      <visual>
-        <origin
-          xyz="0 0 0"
-          rpy="0 0 0" />
-        <geometry>
-          <mesh
-            filename="$(find mason_description)/description/meshes/LeftBracketTop.STL" />
-        </geometry>
-        <material
-          name="">
-          <color
-            rgba="0.4 0.4 0.4 1" />
-        </material>
-      </visual>
-      <collision>
-        <origin
-          xyz="0 0 0"
-          rpy="0 0 0" />
-        <geometry>
-          <mesh
-            filename="$(find mason_description)/description/meshes/LeftBracketTop.STL" />
-        </geometry>
-      </collision>
-    </link>
-    <joint
-      name="LBT_LB"
-      type="fixed">
-      <origin
-        xyz="0.0975000000014027 1.1909568830637 0.120000000000417"
-        rpy="-1.5707963267949 0 0" />
-      <parent
-        link="LeftBar" />
-      <child
-        link="LeftBracketTop" />
-      <axis
-        xyz="0 0 0" />
-    </joint>
-    <link
-      name="LeftBracketBottom">
-      <inertial>
-        <origin
-          xyz="-0.0307068750986306 0.0431985153105867 -6.2978142628678E-07"
-          rpy="0 0 0" />
-        <mass
-          value="0.000214749814862542" />
-        <inertia
-          ixx="5.04014900228218E-07"
-          ixy="1.41838418654998E-07"
-          ixz="-1.26884313983503E-12"
-          iyy="2.49863376560336E-07"
-          iyz="4.06202655988751E-12"
-          izz="5.24669847054166E-07" />
-      </inertial>
-      <visual>
-        <origin
-          xyz="0 0 0"
-          rpy="0 0 0" />
-        <geometry>
-          <mesh
-            filename="$(find mason_description)/description/meshes/LeftBracketBottom.STL" />
-        </geometry>
-        <material
-          name="">
-          <color
-            rgba="0.4 0.4 0.4 1" />
-        </material>
-      </visual>
-      <collision>
-        <origin
-          xyz="0 0 0"
-          rpy="0 0 0" />
-        <geometry>
-          <mesh
-            filename="$(find mason_description)/description/meshes/LeftBracketBottom.STL" />
-        </geometry>
-      </collision>
-    </link>
-    <joint
-      name="LBB_LB"
-      type="fixed">
-      <origin
-        xyz="0.0974999999999891 0.163969013671525 0.12"
-        rpy="-1.5707963267949 0 0" />
-      <parent
-        link="LeftBar" />
-      <child
-        link="LeftBracketBottom" />
-      <axis
-        xyz="0 0 0" />
-    </joint>
-    <link
-      name="WheelHinge1Right">
-      <inertial>
-        <origin
-          xyz="-0.0150182712144393 -0.176153022927531 0.0345338768293388"
-          rpy="0 0 0" />
-        <mass
-          value="0.214742930836365" />
-        <inertia
-          ixx="0.000830775779814993"
-          ixy="-3.28525561723032E-05"
-          ixz="-0.000115730835677916"
-          iyy="0.000823146607327791"
-          iyz="-0.000146137364884107"
-          izz="0.000149954007145533" />
-      </inertial>
-      <visual>
-        <origin
-          xyz="0 0 0"
-          rpy="0 0 0" />
-        <geometry>
-          <mesh
-            filename="$(find mason_description)/description/meshes/WheelHinge1Right.STL" />
-        </geometry>
-        <material
-          name="">
-          <color
-            rgba="0.792156862745098 0.819607843137255 0.933333333333333 1" />
-        </material>
-      </visual>
-      <collision>
-        <origin
-          xyz="0 0 0"
-          rpy="0 0 0" />
-        <geometry>
-          <mesh
-            filename="$(find mason_description)/description/meshes/WheelHinge1Right.STL" />
-        </geometry>
-      </collision>
-    </link>
-    <joint
-      name="gantryVertical"
-      type="prismatic">
-      <origin
-        xyz="-1.34046800536291 -0.272459904837837 0.0227356955196975"
-        rpy="1.5707963267949 0 3.14159265358979" />
-      <parent
-        link="RightBar" />
-      <child
-        link="WheelHinge1Right" />
-      <axis
-        xyz="0 1 0" />
-      <limit
-        lower="-0.4"
-        upper="0.4"
-        effort="100000"
-        velocity="10" />
-    </joint>
-    <link
-      name="Horizontal Bar Bottom">
-      <inertial>
-        <origin
-          xyz="-1.45439216225896E-14 -0.649999999999998 0.175692112504627"
-          rpy="0 0 0" />
-        <mass
-          value="5.55312910017434" />
-        <inertia
-          ixx="0.782838152186632"
-          ixy="-2.04774376725019E-14"
-          ixz="1.10469557216151E-17"
-          iyy="0.00154494115749394"
-          iyz="2.25117904803473E-17"
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