Commit message: integrating odrives (hw intf + xacro)

File: PI/src/mason_description/description/urdf/mason.ros2_control.xacro (robot description, xacro)
@@ -6,5 +6,5 @@
         <hardware>
           <plugin>mason_hardware/MasonInterface</plugin>
-          <param name="device">/dev/ttyACM0</param>
+          <!-- <param name="device">/dev/ttyACM0</param>
           <param name="left_motor_name">motor_left</param>
           <param name="right_motor_name">motor_right</param>
@@ -13,5 +13,6 @@
           <param name="id_left">125</param>
           <param name="id_right">72</param>
-          <param name="id_horizontal">1</param>
+          <param name="id_horizontal">1</param> -->
+          <param name="can">can0</param>
         </hardware>
       </xacro:unless>
@@ -23,4 +24,5 @@
       </xacro:if>
       <joint name="${prefix}motor_horizontal">
+        <param name="node_id">0</param>
         <command_interface name="position">
         </command_interface>
@@ -28,7 +30,12 @@
       </joint>
       <joint name="${prefix}motor_left">
+        <param name="node_id">1</param>
         <command_interface name="position">
         </command_interface>
-        <state_interface name="position"/>>
+        <state_interface name="position"/>
+      </joint>
+      <joint name="${prefix}motor_right">
+        <param name="node_id">2</param>
+        <state_interface name="position"/>
       </joint>
     </ros2_control>
