Commit message: mason test

File: PI/src/mason_description/description/urdf/mason.urdf.xacro (robot description, xacro)
@@ -4,5 +4,5 @@
   <xacro:arg name="slowdown" default="100.0" />
   <xacro:include filename="$(find mason_description)/description/urdf/mason_description.urdf.xacro" />
-  <xacro:include filename="$(find mason_description)/description/urdf/mason.ros2_control.xacro" />
+  <xacro:include filename="$(find mason_description)/description/urdf/mason2.ros2_control.xacro" />
   <xacro:mason />
   <xacro:mason_ros2_control

File: PI/src/mason_description/description/urdf/mason2.ros2_control.xacro (robot description, xacro)
@@ -5,5 +5,5 @@
       <xacro:unless value="${use_mock_hardware}">
         <hardware>
-          <plugin>odrive_ros2_control/ODriveHardwareInterface</plugin>
+          <plugin>odrive_ros2_control_plugin/ODriveHardwareInterface</plugin>
           <param name="can">can0</param>
         </hardware>
@@ -16,4 +16,13 @@
       </xacro:if>
       <joint name="${prefix}motor_horizontal">
+        <param name="node_id">2</param>
+        <command_interface name="position">
+        </command_interface>
+        <command_interface name="velocity">
+        </command_interface>
+        <state_interface name="position"/>
+        <state_interface name="velocity"/>
+      </joint>
+      <joint name="${prefix}motor_left">
         <param name="node_id">0</param>
         <command_interface name="position">
@@ -22,6 +31,7 @@
         </command_interface>
         <state_interface name="position"/>
+        <state_interface name="velocity"/>
       </joint>
-      <joint name="${prefix}motor_left">
+      <joint name="${prefix}motor_right">
         <param name="node_id">1</param>
         <command_interface name="position">
@@ -30,12 +40,5 @@
         </command_interface>
         <state_interface name="position"/>
-      </joint>
-      <joint name="${prefix}motor_right">
-        <param name="node_id">2</param>
-        <command_interface name="position">
-        </command_interface>
-        <command_interface name="velocity">
-        </command_interface>
-        <state_interface name="position"/>
+        <state_interface name="velocity"/>
       </joint>
     </ros2_control>
